Commit message: Second last prax done

File: src/motoman/motoman_sda10f_support/urdf/sda10f_macro.xacro (robot description, xacro)
@@ -1,19 +1,13 @@
 <?xml version="1.0" ?>
-<robot xmlns:xacro="http://ros.org/wiki/xacro">
-     <xacro:include filename="$(find motoman_sda10f_support)/urdf/common_torso_macro.xacro" />
-     <xacro:include filename="$(find motoman_sda10f_support)/urdf/arm_macro.xacro" />
-     <xacro:macro name="motoman_sda10f" params="prefix">
-        <xacro:torso name="torso" prefix="${prefix}torso_"/>
-        <xacro:motoman_arm name="${prefix}arm_left" prefix="${prefix}arm_left_" parent="${prefix}torso_link_b1" reflect="1">
+<robot xmlns:xacro="http://ros.org/wiki/xacro"
+    name="sda10f">
+        <xacro:include filename="$(find motoman_sda10f_support)/urdf/common_torso_macro.xacro" />
+        <xacro:include filename="$(find motoman_sda10f_support)/urdf/arm_macro.xacro" />
+        <xacro:torso name="torso" prefix="torso_"/>
+        <xacro:motoman_arm name="arm_left" prefix="arm_left_" parent="torso_link_b1" reflect="1">
             <origin xyz="0.09996 0.0275 0.32214" rpy="1.57 0 0" />
         </xacro:motoman_arm>
-        <xacro:motoman_arm name="${prefix}arm_right" prefix="${prefix}arm_right_" parent="${prefix}torso_link_b1" reflect="-1">
+        <xacro:motoman_arm name="arm_right" prefix="arm_right_" parent="torso_link_b1" reflect="-1">
             <origin xyz="0.09996 -0.0275 0.32214" rpy="1.57 0 0" />
         </xacro:motoman_arm>
-     </xacro:macro>
-<!-- The following xacro is kept for backwards compatibility, it should not be used -->
-<!-- see: https://github.com/ros-industrial/motoman/issues/166 -->
-     <xacro:macro name="sda10f">
-          <xacro:motoman_sda10f prefix=""/>
-     </xacro:macro>
 </robot>
